File: lab2/Lab2_Solution.sch (EAGLE design)
At the start: 4 parts, among them J1 2.1MMJACKTHM

Commit message: finished lab 2
Parts:
- renumbered SWITCH to U$1
Connections:
- net N$2: now also U$1.2, U$1.4
- net N$3: now also U$1.1, U$1.3
Changed lines of the file:
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@@
 <setting verticaltext="up"/>
 </settings>
-<grid distance="0.1" unitdist="inch" unit="mm" style="lines" multiple="1" display="no" altdistance="0.01" altunitdist="inch" altunit="inch"/>
+<grid distance="0.1" unitdist="inch" unit="inch" style="lines" multiple="1" display="no" altdistance="0.01" altunitdist="inch" altunit="inch"/>
 <layers>
 <layer number="1" name="Top" color="4" fill="1" visible="no" active="no"/>
@@
 <part name="LED1" library="Lab2" deviceset="LED" device="5MM" value="Red"/>
 <part name="R1" library="Lab2" deviceset="RESISTOR" device="AXIAL-0.3" value="330Ohms"/>
-<part name="SWITCH" library="Matt Asaro-Lab2" deviceset="1301" device="1301"/>
+<part name="U$1" library="Matt Asaro-Lab2" deviceset="1301" device="1301"/>
 </parts>
 <sheets>
@@
 <instance part="LED1" gate="G$1" x="35.56" y="53.34" rot="R90"/>
 <instance part="R1" gate="G$1" x="58.42" y="53.34"/>
-<instance part="SWITCH" gate="G$1" x="45.72" y="40.64"/>
+<instance part="U$1" gate="G$1" x="45.72" y="40.64"/>
 </instances>
 <busses>
@@
 <wire x1="63.5" y1="53.34" x2="66.04" y2="53.34" width="0.1524" layer="91"/>
 <wire x1="66.04" y1="53.34" x2="66.04" y2="38.1" width="0.1524" layer="91"/>
+<pinref part="U$1" gate="G$1" pin="4"/>
 <wire x1="66.04" y1="38.1" x2="53.34" y2="38.1" width="0.1524" layer="91"/>
+<pinref part="U$1" gate="G$1" pin="2"/>
 <wire x1="53.34" y1="38.1" x2="53.34" y2="45.72" width="0.1524" layer="91"/>
 </segment>
@@
 <segment>
 <pinref part="J1" gate="G$1" pin="RING"/>
+<pinref part="U$1" gate="G$1" pin="3"/>
 <wire x1="25.4" y1="38.1" x2="38.1" y2="38.1" width="0.1524" layer="91"/>
+<pinref part="U$1" gate="G$1" pin="1"/>
 <wire x1="38.1" y1="38.1" x2="38.1" y2="45.72" width="0.1524" layer="91"/>
 </segment>
