File: lab2/Lab2_Solution.brd (EAGLE design)
At the start: 40.3 x 31.7 mm, 4 parts, among them J1 2.1MMJACKTHM

Commit message: finished lab 2
Parts:
- removed SWITCH: 13011301, Matt Asaro-Lab2:LSH.1301.9315
- added U$1: 13011301, Matt Asaro-Lab2:LSH.1301.9315
Connections:
- net N$2: now also U$1.P$2, U$1.P$4
- net N$3: now also U$1.P$1, U$1.P$3
Routing:
- net N$3: track 0.00 -> 23.2 mm
- net N$2: track 12.5 -> 27.9 mm
Changed lines of the file:
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@@
 <element name="LED1" library="Lab2" package="LED5MM" value="Red" x="30.48" y="22.86"/>
 <element name="R1" library="Lab2" package="AXIAL-0.3" value="330Ohms" x="30.48" y="10.16"/>
-<element name="SWITCH" library="Matt Asaro-Lab2" package="LSH.1301.9315" value="13011301" x="6.35" y="3.81"/>
+<element name="U$1" library="Matt Asaro-Lab2" package="LSH.1301.9315" value="13011301" x="8.89" y="3.81"/>
 </elements>
 <signals>
@@
 <wire x1="31.75" y1="7.62" x2="22.86" y2="7.62" width="0.4064" layer="1"/>
 <wire x1="34.29" y1="10.16" x2="31.75" y2="7.62" width="0.4064" layer="1"/>
+<contactref element="U$1" pad="P$4"/>
+<contactref element="U$1" pad="P$2"/>
+<wire x1="18.89" y1="3.81" x2="18.89" y2="8.31" width="0.4064" layer="1"/>
+<wire x1="22.86" y1="7.62" x2="22.86" y2="11.43" width="0.4064" layer="1"/>
+<wire x1="22.86" y1="11.43" x2="18.89" y2="11.43" width="0.4064" layer="1"/>
+<wire x1="18.89" y1="11.43" x2="18.89" y2="8.31" width="0.4064" layer="1"/>
 </signal>
 <signal name="N$4">
@@
 <signal name="N$3">
 <contactref element="J1" pad="RING"/>
+<contactref element="U$1" pad="P$3"/>
+<contactref element="U$1" pad="P$1"/>
+<wire x1="8.89" y1="3.81" x2="8.89" y2="8.31" width="0.4064" layer="1"/>
+<wire x1="11.01" y1="24.865" x2="8.89" y2="24.865" width="0.4064" layer="1"/>
+<wire x1="8.89" y1="24.865" x2="8.89" y2="8.31" width="0.4064" layer="1"/>
 </signal>
 </signals>

Commit message: finished
Parts:
- added U$2: (no value), Matt Asaro-Lab2:UCSD_LOGO
Changed lines of the file:
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@@
 <element name="R1" library="Lab2" package="AXIAL-0.3" value="330Ohms" x="30.48" y="10.16"/>
 <element name="U$1" library="Matt Asaro-Lab2" package="LSH.1301.9315" value="13011301" x="8.89" y="3.81"/>
+<element name="U$2" library="Matt Asaro-Lab2" package="UCSD_LOGO" value="" x="30.48" y="29.21"/>
 </elements>
 <signals>
