File: lab5/working/lab5.sch (EAGLE design)
At the start: 13 parts, among them U1 ATMEGA128RFA1, Y1 16MHz

Commit message: updated lab5.sch
Parts:
- added C9: 0.1 uF, Lab5:C-USC0805
- added J1: ISP, Lab5:AVR_SPI_PRG_6NS
- added JP1, JP2: FTDI_BASICPTH, Lab5:FTDI_BASICPTH
- added LED1, LED2: GREEN, Lab5:LEDCHIP-LED0805
- added R2, R3: 330, Lab5:R-US_R0805
- added S1: SWITCH-MOMENTARY-2SMD, Lab5:SWITCH-MOMENTARY-2SMD
Connections:
- new net N$8: LED1.A, R2.1
- new net N$9: LED2.A, R3.1
- net GND: now also J1.6, JP1.6, JP2.6, LED1.C, LED2.C, S1.2
- net MISO: now also J1.1
- net MOSI: now also J1.4
- net PB6: now also R2.2
- net PB7: now also R3.2
- net RESET: now also C9.2, J1.5, S1.1
- net RX0: now also JP1.3
- net RX1: now also JP2.3
- net SCK: now also J1.3
- net TX0: now also C9.1, JP1.1, JP1.2
- net TX1: now also JP2.2
Changed lines of the file:
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@@
 <part name="GND9" library="Lab5" deviceset="GND" device=""/>
 <part name="A1" library="Lab5" deviceset="ANTENNA2" device="SMD5"/>
+<part name="LED1" library="Lab5" deviceset="LED" device="CHIP-LED0805" value="GREEN"/>
+<part name="LED2" library="Lab5" deviceset="LED" device="CHIP-LED0805" value="GREEN"/>
+<part name="R2" library="Lab5" deviceset="R-US_" device="R0805" value="330"/>
+<part name="R3" library="Lab5" deviceset="R-US_" device="R0805" value="330"/>
+<part name="GND10" library="Lab5" deviceset="GND" device=""/>
+<part name="GND11" library="Lab5" deviceset="GND" device=""/>
+<part name="JP1" library="Lab5" deviceset="FTDI_BASIC" device="PTH"/>
+<part name="GND12" library="Lab5" deviceset="GND" device=""/>
+<part name="JP2" library="Lab5" deviceset="FTDI_BASIC" device="PTH"/>
+<part name="C9" library="Lab5" deviceset="C-US" device="C0805" value="0.1 uF"/>
+<part name="S1" library="Lab5" deviceset="SWITCH-MOMENTARY-2" device="SMD" value=""/>
+<part name="GND13" library="Lab5" deviceset="GND" device=""/>
+<part name="GND14" library="Lab5" deviceset="GND" device=""/>
+<part name="J1" library="Lab5" deviceset="AVR_SPI_PRG_6" device="NS" value="ISP"/>
+<part name="GND15" library="Lab5" deviceset="GND" device=""/>
 </parts>
 <sheets>
@@
 <instance part="GND9" gate="1" x="48.26" y="-20.32"/>
 <instance part="A1" gate="G$1" x="53.34" y="10.16"/>
+<instance part="LED1" gate="G$1" x="-127" y="-55.88" rot="MR0"/>
+<instance part="LED2" gate="G$1" x="-111.76" y="-55.88" rot="MR0"/>
+<instance part="R2" gate="G$1" x="-127" y="-43.18" rot="R90"/>
+<instance part="R3" gate="G$1" x="-111.76" y="-43.18" rot="R90"/>
+<instance part="GND10" gate="1" x="-127" y="-66.04"/>
+<instance part="GND11" gate="1" x="-111.76" y="-66.04"/>
+<instance part="JP1" gate="G$1" x="17.78" y="55.88" rot="MR180"/>
+<instance part="GND12" gate="1" x="30.48" y="40.64"/>
+<instance part="JP2" gate="G$1" x="-10.16" y="55.88" rot="MR180"/>
+<instance part="C9" gate="G$1" x="38.1" y="60.96" rot="R90"/>
+<instance part="S1" gate="G$1" x="68.58" y="43.18" rot="R270"/>
+<instance part="GND13" gate="1" x="68.58" y="27.94"/>
+<instance part="GND14" gate="1" x="-2.54" y="40.64"/>
+<instance part="J1" gate="G$1" x="22.86" y="25.4"/>
+<instance part="GND15" gate="1" x="38.1" y="12.7"/>
 </instances>
 <busses>
@@
 <wire x1="48.26" y1="-12.7" x2="48.26" y2="-17.78" width="0.1524" layer="91"/>
 </segment>
+<segment>
+<pinref part="LED1" gate="G$1" pin="C"/>
+<wire x1="-127" y1="-60.96" x2="-127" y2="-63.5" width="0.1524" layer="91"/>
+<pinref part="GND10" gate="1" pin="GND"/>
+</segment>
+<segment>
+<pinref part="LED2" gate="G$1" pin="C"/>
+<wire x1="-111.76" y1="-60.96" x2="-111.76" y2="-63.5" width="0.1524" layer="91"/>
+<pinref part="GND11" gate="1" pin="GND"/>
+</segment>
+<segment>
+<pinref part="JP1" gate="G$1" pin="6"/>
+<wire x1="22.86" y1="48.26" x2="30.48" y2="48.26" width="0.1524" layer="91"/>
+<pinref part="GND12" gate="1" pin="GND"/>
+<wire x1="30.48" y1="48.26" x2="30.48" y2="43.18" width="0.1524" layer="91"/>
+</segment>
+<segment>
+<pinref part="S1" gate="G$1" pin="2"/>
+<pinref part="GND13" gate="1" pin="GND"/>
+<wire x1="68.58" y1="38.1" x2="68.58" y2="30.48" width="0.1524" layer="91"/>
+</segment>
+<segment>
+<pinref part="JP2" gate="G$1" pin="6"/>
+<wire x1="-5.08" y1="48.26" x2="-2.54" y2="48.26" width="0.1524" layer="91"/>
+<wire x1="-2.54" y1="48.26" x2="-2.54" y2="43.18" width="0.1524" layer="91"/>
+<pinref part="GND14" gate="1" pin="GND"/>
+</segment>
+<segment>
+<pinref part="J1" gate="G$1" pin="6"/>
+<wire x1="33.02" y1="22.86" x2="38.1" y2="22.86" width="0.1524" layer="91"/>
+<pinref part="GND15" gate="1" pin="GND"/>
+<wire x1="38.1" y1="22.86" x2="38.1" y2="15.24" width="0.1524" layer="91"/>
+</segment>
 </net>
 <net name="A7" class="0">
@@
 <pinref part="R1" gate="G$1" pin="1"/>
 <wire x1="-12.7" y1="-7.62" x2="-12.7" y2="-5.08" width="0.1524" layer="91"/>
-<label x="-7.62" y="-7.62" size="1.27" layer="95"/>
+<label x="-7.62" y="-7.62" size="1.27" layer="95" xref="yes"/>
 <wire x1="-12.7" y1="-7.62" x2="-7.62" y2="-7.62" width="0.1524" layer="91"/>
 <junction x="-12.7" y="-7.62"/>
+</segment>
+<segment>
+<pinref part="C9" gate="G$1" pin="2"/>
+<wire x1="43.18" y1="60.96" x2="45.72" y2="60.96" width="0.1524" layer="91"/>
+<label x="45.72" y="60.96" size="1.27" layer="95" xref="yes"/>
+</segment>
+<segment>
+<pinref part="S1" gate="G$1" pin="1"/>
+<wire x1="68.58" y1="48.26" x2="68.58" y2="53.34" width="0.1524" layer="91"/>
+<wire x1="68.58" y1="53.34" x2="73.66" y2="53.34" width="0.1524" layer="91"/>
+<label x="73.66" y="53.34" size="1.27" layer="95" xref="yes"/>
+</segment>
+<segment>
+<pinref part="J1" gate="G$1" pin="5"/>
+<wire x1="15.24" y1="22.86" x2="7.62" y2="22.86" width="0.1524" layer="91"/>
+<label x="7.62" y="22.86" size="1.27" layer="95" rot="R180" xref="yes"/>
 </segment>
 </net>
@@
 <label x="-88.9" y="-48.26" size="1.27" layer="95" rot="R180" xref="yes"/>
 </segment>
+<segment>
+<pinref part="JP1" gate="G$1" pin="1"/>
+<pinref part="C9" gate="G$1" pin="1"/>
+<wire x1="22.86" y1="60.96" x2="35.56" y2="60.96" width="0.1524" layer="91"/>
+</segment>
+<segment>
+<pinref part="JP1" gate="G$1" pin="2"/>
+<wire x1="22.86" y1="58.42" x2="25.4" y2="58.42" width="0.1524" layer="91"/>
+<label x="25.4" y="58.42" size="1.27" layer="95" xref="yes"/>
+</segment>
 </net>
 <net name="RX0" class="0">
@@
 <label x="-88.9" y="-45.72" size="1.27" layer="95" rot="R180" xref="yes"/>
 </segment>
+<segment>
+<pinref part="JP1" gate="G$1" pin="3"/>
+<wire x1="22.86" y1="55.88" x2="25.4" y2="55.88" width="0.1524" layer="91"/>
+<label x="25.4" y="55.88" size="1.27" layer="95" xref="yes"/>
+</segment>
 </net>
 <net name="PD7" class="0">
@@
 <label x="-88.9" y="-30.48" size="1.27" layer="95" rot="R180" xref="yes"/>
 </segment>
+<segment>
+<pinref part="JP2" gate="G$1" pin="2"/>
+<wire x1="-5.08" y1="58.42" x2="-2.54" y2="58.42" width="0.1524" layer="91"/>
+<label x="-2.54" y="58.42" size="1.27" layer="95" xref="yes"/>
+</segment>
 </net>
 <net name="RX1" class="0">
@@
 <label x="-88.9" y="-27.94" size="1.27" layer="95" rot="R180" xref="yes"/>
 </segment>
+<segment>
+<pinref part="JP2" gate="G$1" pin="3"/>
+<wire x1="-5.08" y1="55.88" x2="-2.54" y2="55.88" width="0.1524" layer="91"/>
+<label x="-2.54" y="55.88" size="1.27" layer="95" xref="yes"/>
+</segment>
 </net>
 <net name="SDA" class="0">
@@
 <label x="-88.9" y="-17.78" size="1.27" layer="95" rot="R180" xref="yes"/>
 </segment>
+<segment>
+<pinref part="R3" gate="G$1" pin="2"/>
+<wire x1="-111.76" y1="-38.1" x2="-111.76" y2="-30.48" width="0.1524" layer="91"/>
+<label x="-132.08" y="-30.48" size="1.27" layer="95" rot="MR0" xref="yes"/>
+<wire x1="-111.76" y1="-30.48" x2="-132.08" y2="-30.48" width="0.1524" layer="91"/>
+</segment>
 </net>
 <net name="PB6" class="0">
@@
 <label x="-88.9" y="-15.24" size="1.27" layer="95" rot="R180" xref="yes"/>
 </segment>
+<segment>
+<pinref part="R2" gate="G$1" pin="2"/>
+<wire x1="-127" y1="-38.1" x2="-127" y2="-35.56" width="0.1524" layer="91"/>
+<label x="-132.08" y="-35.56" size="1.27" layer="95" rot="MR0" xref="yes"/>
+<wire x1="-127" y1="-35.56" x2="-132.08" y2="-35.56" width="0.1524" layer="91"/>
+</segment>
 </net>
 <net name="PB5" class="0">
@@
 <label x="-88.9" y="-7.62" size="1.27" layer="95" rot="R180" xref="yes"/>
 </segment>
+<segment>
+<pinref part="J1" gate="G$1" pin="1"/>
+<wire x1="15.24" y1="27.94" x2="7.62" y2="27.94" width="0.1524" layer="91"/>
+<label x="7.62" y="27.94" size="1.27" layer="95" rot="R180" xref="yes"/>
+</segment>
 </net>
 <net name="MOSI" class="0">
@@
 <label x="-88.9" y="-5.08" size="1.27" layer="95" rot="R180" xref="yes"/>
 </segment>
+<segment>
+<pinref part="J1" gate="G$1" pin="4"/>
+<wire x1="33.02" y1="25.4" x2="38.1" y2="25.4" width="0.1524" layer="91"/>
+<label x="38.1" y="25.4" size="1.27" layer="95" xref="yes"/>
+</segment>
 </net>
 <net name="SCK" class="0">
@@
 <wire x1="-83.82" y1="-2.54" x2="-88.9" y2="-2.54" width="0.1524" layer="91"/>
 <label x="-88.9" y="-2.54" size="1.27" layer="95" rot="R180" xref="yes"/>
+</segment>
+<segment>
+<pinref part="J1" gate="G$1" pin="3"/>
+<wire x1="15.24" y1="25.4" x2="7.62" y2="25.4" width="0.1524" layer="91"/>
+<label x="7.62" y="25.4" size="1.27" layer="95" rot="R180" xref="yes"/>
 </segment>
 </net>
@@
 </segment>
 </net>
+<net name="N$8" class="0">
+<segment>
+<pinref part="R2" gate="G$1" pin="1"/>
+<pinref part="LED1" gate="G$1" pin="A"/>
+<wire x1="-127" y1="-48.26" x2="-127" y2="-53.34" width="0.1524" layer="91"/>
+</segment>
+</net>
+<net name="N$9" class="0">
+<segment>
+<pinref part="R3" gate="G$1" pin="1"/>
+<pinref part="LED2" gate="G$1" pin="A"/>
+<wire x1="-111.76" y1="-48.26" x2="-111.76" y2="-53.34" width="0.1524" layer="91"/>
+</segment>
+</net>

Commit message: added power connectors
Parts:
- added C10, C11: 1 uF, Lab5:C-USC0805
- added JP3: (no value), Lab5:M02PTH
- added LED3: RED, Lab5:LEDCHIP-LED0805
- added R4: 1k, Lab5:R-US_R0805
- added S2: (no value), Lab5:SWITCH-SPDTPTH
- added U$1: LP3985IM5-3.0, Lab5:LP3985IM5-3.0
Connections:
- new net N$10: C11.2, S2.O, U$1.EN, U$1.IN
- new net N$6: LED3.A, R4.1
- new net N$7: JP3.2, S2.P
- net 3.3V: now also C10.2, R4.2, U$1.OUT
- net GND: now also C10.1, C11.1, JP3.1, LED3.C, U$1.GND
Changed lines of the file:
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@@
 <part name="J1" library="Lab5" deviceset="AVR_SPI_PRG_6" device="NS" value="ISP"/>
 <part name="GND15" library="Lab5" deviceset="GND" device=""/>
+<part name="JP3" library="Lab5" deviceset="M02" device="PTH"/>
+<part name="S2" library="Lab5" deviceset="SWITCH-SPDT" device="PTH"/>
+<part name="U$1" library="Lab5" deviceset="LP3985IM5-3.0" device=""/>
+<part name="GND16" library="Lab5" deviceset="GND" device=""/>
+<part name="GND17" library="Lab5" deviceset="GND" device=""/>
+<part name="C10" library="Lab5" deviceset="C-US" device="C0805" value="1 uF"/>
+<part name="C11" library="Lab5" deviceset="C-US" device="C0805" value="1 uF"/>
+<part name="GND18" library="Lab5" deviceset="GND" device=""/>
+<part name="GND19" library="Lab5" deviceset="GND" device=""/>
+<part name="P+3" library="Lab5" deviceset="3.3V" device="" value="3V"/>
+<part name="LED3" library="Lab5" deviceset="LED" device="CHIP-LED0805" value="RED"/>
+<part name="GND20" library="Lab5" deviceset="GND" device=""/>
+<part name="R4" library="Lab5" deviceset="R-US_" device="R0805" value="1k"/>
 </parts>
 <sheets>
@@
 <instance part="J1" gate="G$1" x="22.86" y="25.4"/>
 <instance part="GND15" gate="1" x="38.1" y="12.7"/>
+<instance part="JP3" gate="G$1" x="-124.46" y="38.1"/>
+<instance part="S2" gate="1" x="-106.68" y="50.8"/>
+<instance part="U$1" gate="G$1" x="-76.2" y="40.64"/>
+<instance part="GND16" gate="1" x="-114.3" y="27.94"/>
+<instance part="GND17" gate="1" x="-81.28" y="30.48"/>
+<instance part="C10" gate="G$1" x="-45.72" y="43.18" rot="R180"/>
+<instance part="C11" gate="G$1" x="-91.44" y="40.64" rot="R180"/>
+<instance part="GND18" gate="1" x="-91.44" y="30.48"/>
+<instance part="GND19" gate="1" x="-45.72" y="30.48"/>
+<instance part="P+3" gate="G$1" x="-53.34" y="63.5"/>
+<instance part="LED3" gate="G$1" x="-30.48" y="43.18" rot="MR0"/>
+<instance part="GND20" gate="1" x="-30.48" y="30.48"/>
+<instance part="R4" gate="G$1" x="-38.1" y="53.34" rot="R180"/>
 </instances>
 <busses>
@@
 <wire x1="38.1" y1="22.86" x2="38.1" y2="15.24" width="0.1524" layer="91"/>
 </segment>
+<segment>
+<pinref part="JP3" gate="G$1" pin="1"/>
+<wire x1="-116.84" y1="38.1" x2="-114.3" y2="38.1" width="0.1524" layer="91"/>
+<pinref part="GND16" gate="1" pin="GND"/>
+<wire x1="-114.3" y1="38.1" x2="-114.3" y2="30.48" width="0.1524" layer="91"/>
+</segment>
+<segment>
+<pinref part="C11" gate="G$1" pin="1"/>
+<pinref part="GND18" gate="1" pin="GND"/>
+<wire x1="-91.44" y1="38.1" x2="-91.44" y2="33.02" width="0.1524" layer="91"/>
+</segment>
+<segment>
+<pinref part="U$1" gate="G$1" pin="GND"/>
+<wire x1="-78.74" y1="48.26" x2="-81.28" y2="48.26" width="0.1524" layer="91"/>
+<pinref part="GND17" gate="1" pin="GND"/>
+<wire x1="-81.28" y1="48.26" x2="-81.28" y2="33.02" width="0.1524" layer="91"/>
+</segment>
+<segment>
+<pinref part="C10" gate="G$1" pin="1"/>
+<pinref part="GND19" gate="1" pin="GND"/>
+<wire x1="-45.72" y1="40.64" x2="-45.72" y2="33.02" width="0.1524" layer="91"/>
+</segment>
+<segment>
+<pinref part="LED3" gate="G$1" pin="C"/>
+<pinref part="GND20" gate="1" pin="GND"/>
+<wire x1="-30.48" y1="38.1" x2="-30.48" y2="33.02" width="0.1524" layer="91"/>
+</segment>
 </net>
 <net name="A7" class="0">
@@
 <wire x1="-22.86" y1="0" x2="-22.86" y2="7.62" width="0.1524" layer="91"/>
 <junction x="-22.86" y="0"/>
+</segment>
+<segment>
+<pinref part="U$1" gate="G$1" pin="OUT"/>
+<wire x1="-55.88" y1="53.34" x2="-53.34" y2="53.34" width="0.1524" layer="91"/>
+<pinref part="P+3" gate="G$1" pin="3.3V"/>
+<wire x1="-53.34" y1="63.5" x2="-53.34" y2="53.34" width="0.1524" layer="91"/>
+<wire x1="-53.34" y1="53.34" x2="-45.72" y2="53.34" width="0.1524" layer="91"/>
+<junction x="-53.34" y="53.34"/>
+<pinref part="C10" gate="G$1" pin="2"/>
+<wire x1="-45.72" y1="53.34" x2="-45.72" y2="48.26" width="0.1524" layer="91"/>
+<pinref part="R4" gate="G$1" pin="2"/>
+<wire x1="-45.72" y1="53.34" x2="-43.18" y2="53.34" width="0.1524" layer="91"/>
+<junction x="-45.72" y="53.34"/>
 </segment>
 </net>
@@
 </segment>
 </net>
+<net name="N$7" class="0">
+<segment>
+<pinref part="JP3" gate="G$1" pin="2"/>
+<wire x1="-116.84" y1="40.64" x2="-109.22" y2="40.64" width="0.1524" layer="91"/>
+<wire x1="-109.22" y1="40.64" x2="-109.22" y2="50.8" width="0.1524" layer="91"/>
+<pinref part="S2" gate="1" pin="P"/>
+</segment>
+</net>
+<net name="N$10" class="0">
+<segment>
+<pinref part="S2" gate="1" pin="O"/>
+<pinref part="U$1" gate="G$1" pin="IN"/>
+<wire x1="-101.6" y1="53.34" x2="-91.44" y2="53.34" width="0.1524" layer="91"/>
+<wire x1="-91.44" y1="53.34" x2="-83.82" y2="53.34" width="0.1524" layer="91"/>
+<wire x1="-83.82" y1="53.34" x2="-78.74" y2="53.34" width="0.1524" layer="91"/>
+<wire x1="-83.82" y1="53.34" x2="-83.82" y2="43.18" width="0.1524" layer="91"/>
+<junction x="-83.82" y="53.34"/>
+<pinref part="U$1" gate="G$1" pin="EN"/>
+<wire x1="-83.82" y1="43.18" x2="-78.74" y2="43.18" width="0.1524" layer="91"/>
+<pinref part="C11" gate="G$1" pin="2"/>
+<wire x1="-91.44" y1="53.34" x2="-91.44" y2="45.72" width="0.1524" layer="91"/>
+<junction x="-91.44" y="53.34"/>
+</segment>
+</net>
+<net name="N$6" class="0">
+<segment>
+<pinref part="R4" gate="G$1" pin="1"/>
+<wire x1="-33.02" y1="53.34" x2="-30.48" y2="53.34" width="0.1524" layer="91"/>
+<pinref part="LED3" gate="G$1" pin="A"/>
+<wire x1="-30.48" y1="53.34" x2="-30.48" y2="45.72" width="0.1524" layer="91"/>
+</segment>
+</net>
