File: lab5/working/lab5.sch (EAGLE design)
At the start: 53 parts, among them J1 ISP, U1 ATMEGA128RFA1, Y1 16MHz

Commit message: updated schematic to use Kirt library
Parts:
- removed C5, C7: JUMP, Lab5:C-USC0805
- removed U$10, U$13, U$4, U$7: BAS16WS, lab4:BAS16WS
- removed U$11, U$14, U$5, U$8: SI2302CDS, lab4:SI2302CDS
- removed U$12, U$3, U$6, U$9: RCL0805, lab4:RCL0805
- added D1, D2, D3, D4: DIODE, Kirt-Lab4:DIODE
- added Q1, Q2, Q3, Q4: FET, Kirt-Lab4:FET
- added R10, R7, R8, R9: 10k, Lab5:R-US_R0805
Connections:
- removed net N$32: JP4.1, U$4.P$2, U$5.D3
- removed net N$5: B1.OUT1, C5.2
- net GND: now also Q1.P$2, Q2.P$2, Q3.P$2, Q4.P$2, R10.1, R7.1, R8.1, R9.1; no longer U$11.S2, U$12.P$2, U$14.S2, U$3.P$2, U$5.S2, U$6.P$2, U$8.S2, U$9.P$2
- net N$12: now also D3.P$2, JP4.1, Q4.P$3; no longer JP5.1, U$7.P$2, U$8.D3
- net N$15: now also D2.P$2, JP5.1, Q3.P$3; no longer JP6.1, U$10.P$2, U$11.D3
- net N$16: now also D4.P$2, Q1.P$3; no longer U$13.P$2, U$14.D3
- net N$17: now also B1.OUT2; no longer C7.2
- net N$18: now also B1.OUT1; no longer C5.1
- net N$3: now also D1.P$2, JP6.1, Q2.P$3; no longer B1.OUT2, C7.1
- net PB5: now also Q1.P$1, R7.2; no longer U$12.P$1, U$14.G1
- net PE3: now also Q3.P$1, R9.2; no longer U$6.P$1, U$8.G1
- net PE4: now also Q4.P$1, R10.2; no longer U$3.P$1, U$5.G1
- net PE5: now also Q2.P$1, R8.2; no longer U$11.G1, U$9.P$1
- net VBAT: now also D1.P$1, D2.P$1, D3.P$1, D4.P$1; no longer U$10.P$1, U$13.P$1, U$4.P$1, U$7.P$1

Commit message: grounded CLKI on microcontroller
Connections:
- net GND: now also U1.CLKI
Changed lines of the file:
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@@
 <part name="R10" library="Lab5" deviceset="R-US_" device="R0805" value="10k"/>
 <part name="Q4" library="Kirt-Lab4" deviceset="FET" device=""/>
+<part name="GND30" library="Lab5" deviceset="GND" device=""/>
 </parts>
 <sheets>
@@
 <instance part="R10" gate="G$1" x="-83.82" y="-121.92" rot="R180"/>
 <instance part="Q4" gate="G$1" x="-73.66" y="-96.52"/>
+<instance part="GND30" gate="1" x="63.5" y="-73.66"/>
 </instances>
 <busses>
@@
 <wire x1="-73.66" y1="-107.95" x2="-73.66" y2="-121.92" width="0.1524" layer="91"/>
 </segment>
+<segment>
+<pinref part="U1" gate="G$1" pin="CLKI"/>
+<wire x1="58.42" y1="-68.58" x2="63.5" y2="-68.58" width="0.1524" layer="91"/>
+<pinref part="GND30" gate="1" pin="GND"/>
+<wire x1="63.5" y1="-68.58" x2="63.5" y2="-71.12" width="0.1524" layer="91"/>
+</segment>
 </net>

Commit message: added 2nd cap
Parts:
- added C5: 1 uF, Lab5:C-USC0805
Connections:
- net 3.3V: now also C5.2
- net GND: now also C5.1
Changed lines of the file:
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@@
 <part name="Q4" library="Kirt-Lab4" deviceset="FET" device=""/>
 <part name="GND30" library="Lab5" deviceset="GND" device=""/>
+<part name="P+7" library="Lab5" deviceset="3.3V" device="" value="3V"/>
+<part name="C5" library="Lab5" deviceset="C-US" device="C0805" value="1 uF"/>
+<part name="GND31" library="Lab5" deviceset="GND" device=""/>
 </parts>
 <sheets>
@@
 <instance part="Q4" gate="G$1" x="-73.66" y="-96.52"/>
 <instance part="GND30" gate="1" x="63.5" y="-73.66"/>
+<instance part="P+7" gate="G$1" x="-40.64" y="-27.94"/>
+<instance part="C5" gate="G$1" x="-40.64" y="-35.56" rot="R180"/>
+<instance part="GND31" gate="1" x="-40.64" y="-43.18"/>
 </instances>
 <busses>
@@
 <pinref part="GND30" gate="1" pin="GND"/>
 <wire x1="63.5" y1="-68.58" x2="63.5" y2="-71.12" width="0.1524" layer="91"/>
+</segment>
+<segment>
+<pinref part="C5" gate="G$1" pin="1"/>
+<pinref part="GND31" gate="1" pin="GND"/>
+<wire x1="-40.64" y1="-38.1" x2="-40.64" y2="-40.64" width="0.1524" layer="91"/>
 </segment>
 </net>
@@
 <wire x1="-22.86" y1="-27.94" x2="-22.86" y2="-30.48" width="0.1524" layer="91"/>
 </segment>
-</net>
+<segment>
+<pinref part="P+7" gate="G$1" pin="3.3V"/>
+<pinref part="C5" gate="G$1" pin="2"/>
+<wire x1="-40.64" y1="-27.94" x2="-40.64" y2="-30.48" width="0.1524" layer="91"/>
+</segment>
+</net>

Commit message: fixed resistor values according to piazza post from Jorge and schematic review feedback
Parts:
- R2, R3: value 300 -> 270
- R4: value 1k -> 680
Changed lines of the file:
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@@
 <part name="LED1" library="Lab5" deviceset="LED" device="CHIP-LED0805" value="GREEN"/>
 <part name="LED2" library="Lab5" deviceset="LED" device="CHIP-LED0805" value="GREEN"/>
-<part name="R2" library="Lab5" deviceset="R-US_" device="R0805" value="300"/>
-<part name="R3" library="Lab5" deviceset="R-US_" device="R0805" value="300"/>
+<part name="R2" library="Lab5" deviceset="R-US_" device="R0805" value="270"/>
+<part name="R3" library="Lab5" deviceset="R-US_" device="R0805" value="270"/>
 <part name="GND10" library="Lab5" deviceset="GND" device=""/>
 <part name="GND11" library="Lab5" deviceset="GND" device=""/>
@@
 <part name="LED3" library="Lab5" deviceset="LED" device="CHIP-LED0805" value="RED"/>
 <part name="GND20" library="Lab5" deviceset="GND" device=""/>
-<part name="R4" library="Lab5" deviceset="R-US_" device="R0805" value="1k"/>
+<part name="R4" library="Lab5" deviceset="R-US_" device="R0805" value="680"/>
 <part name="U$2" library="lab4" deviceset="LSM9DS0" device="MAIN"/>
 <part name="P+4" library="Lab5" deviceset="3.3V" device="" value="3V"/>
@@
 <instance part="C15" gate="G$1" x="-147.32" y="114.3" rot="R180"/>
 <instance part="GND23" gate="1" x="-157.48" y="127" rot="R180"/>
-<instance part="GND24" gate="1" x="-203.2" y="43.18"/>
+<instance part="GND24" gate="1" x="-220.98" y="58.42"/>
 <instance part="R5" gate="G$1" x="-215.9" y="83.82" rot="R180"/>
 <instance part="R6" gate="G$1" x="-215.9" y="91.44" rot="R180"/>
@@
 <pinref part="U$2" gate="IMU" pin="P$22"/>
 <wire x1="-198.12" y1="68.58" x2="-198.12" y2="73.66" width="0.1524" layer="91"/>
-<wire x1="-198.12" y1="73.66" x2="-203.2" y2="73.66" width="0.1524" layer="91"/>
+<wire x1="-198.12" y1="73.66" x2="-220.98" y2="73.66" width="0.1524" layer="91"/>
 <junction x="-198.12" y="73.66"/>
-<wire x1="-203.2" y1="73.66" x2="-203.2" y2="45.72" width="0.1524" layer="91"/>
+<wire x1="-220.98" y1="73.66" x2="-220.98" y2="60.96" width="0.1524" layer="91"/>
 <pinref part="GND24" gate="1" pin="GND"/>
 </segment>
